File: PCB/SofleHeavy.sch (KiCad schematic (older format))
At the start: 104 parts, among them J1 LED, J2 4PIN, J3 OLED, J4 USB_C_Receptacle_USB2.0, P1 i2c_pin, P2 i2c_pin, SW1 SW_PUSH, SW10 SW_PUSH, SW11 SW_PUSH, SW12 SW_PUSH, SW13 SW_PUSH, SW14 SW_PUSH, SW15 SW_PUSH, SW16 SW_PUSH, SW17 SW_PUSH, SW18 SW_PUSH, SW19 SW_PUSH, SW2 SW_PUSH, SW20 SW_PUSH, SW21 SW_PUSH, SW22 SW_PUSH, SW23 SW_PUSH, SW24 SW_PUSH, SW25 Rotary_Encoder_Switch, SW26 SW_PUSH, SW27 SW_PUSH, SW28 SW_PUSH, SW29 SW_PUSH, SW3 SW_PUSH, SW30 SW_PUSH, SW4 SW_PUSH, SW5 SW_PUSH, SW6 SW_PUSH, SW7 SW_PUSH, SW8 SW_PUSH, SW9 SW_PUSH, U1 ATmega32U4-AU, Y1 Crystal

Commit message: Started PCB redux
Parts:
- C1, C2, C3, C4, C5, C6, C7, C8: footprint (none) -> Capacitor_SMD:C_0805_2012Metric_Pad1.18x1.45mm_HandSolder
- F1: footprint (none) -> Fuse:Fuse_0603_1608Metric
- FB1: footprint (none) -> Inductor_SMD:L_0201_0603Metric
- J4: footprint (none) -> Connector_USB:USB_C_Receptacle_HRO_TYPE-C-31-M-12
- R1, R2, R3, R4, R5, R6, R7, R8: footprint (none) -> Resistor_SMD:R_0201_0603Metric
- Y1: footprint (none) -> Crystal:Crystal_SMD_3225-4Pin_3.2x2.5mm_HandSoldering
Changed lines of the file:
@@
 F 0 "C1" H 1242 1496 50  0000 L CNN
 F 1 "0.1uF" H 1242 1405 50  0000 L CNN
-F 2 "" H 1150 1450 50  0001 C CNN
+F 2 "Capacitor_SMD:C_0805_2012Metric_Pad1.18x1.45mm_HandSolder" H 1150 1450 50  0001 C CNN
 F 3 "~" H 1150 1450 50  0001 C CNN
 	1    1150 1450
@@
 F 0 "C2" H 1642 1496 50  0000 L CNN
 F 1 "0.1uF" H 1642 1405 50  0000 L CNN
-F 2 "" H 1550 1450 50  0001 C CNN
+F 2 "Capacitor_SMD:C_0805_2012Metric_Pad1.18x1.45mm_HandSolder" H 1550 1450 50  0001 C CNN
 F 3 "~" H 1550 1450 50  0001 C CNN
 	1    1550 1450
@@
 F 0 "C3" H 2042 1496 50  0000 L CNN
 F 1 "0.1uF" H 2042 1405 50  0000 L CNN
-F 2 "" H 1950 1450 50  0001 C CNN
+F 2 "Capacitor_SMD:C_0805_2012Metric_Pad1.18x1.45mm_HandSolder" H 1950 1450 50  0001 C CNN
 F 3 "~" H 1950 1450 50  0001 C CNN
 	1    1950 1450
@@
 F 0 "C4" H 2442 1496 50  0000 L CNN
 F 1 "0.1uF" H 2442 1405 50  0000 L CNN
-F 2 "" H 2350 1450 50  0001 C CNN
+F 2 "Capacitor_SMD:C_0805_2012Metric_Pad1.18x1.45mm_HandSolder" H 2350 1450 50  0001 C CNN
 F 3 "~" H 2350 1450 50  0001 C CNN
 	1    2350 1450
@@
 F 0 "C5" V 2750 2950 50  0000 C CNN
 F 1 "0.1uF" V 2750 2750 50  0000 C CNN
-F 2 "" H 2900 2850 50  0001 C CNN
+F 2 "Capacitor_SMD:C_0805_2012Metric_Pad1.18x1.45mm_HandSolder" H 2900 2850 50  0001 C CNN
 F 3 "~" H 2900 2850 50  0001 C CNN
 	1    2900 2850
@@
 F 0 "R3" V 2750 2500 50  0000 C CNN
 F 1 "22" V 2750 2650 50  0000 C CNN
-F 2 "" V 2890 2540 50  0001 C CNN
+F 2 "Resistor_SMD:R_0201_0603Metric" V 2890 2540 50  0001 C CNN
 F 3 "~" H 2850 2550 50  0001 C CNN
 	1    2850 2550
@@
 F 0 "R4" V 2950 2600 50  0000 C CNN
 F 1 "22" V 2950 2750 50  0000 C CNN
-F 2 "" V 2890 2640 50  0001 C CNN
+F 2 "Resistor_SMD:R_0201_0603Metric" V 2890 2640 50  0001 C CNN
 F 3 "~" H 2850 2650 50  0001 C CNN
 	1    2850 2650
@@
 F 0 "Y1" V 2350 2100 50  0000 L CNN
 F 1 "Crystal" V 2250 2050 50  0000 L CNN
-F 2 "" H 2300 2000 50  0001 C CNN
+F 2 "Crystal:Crystal_SMD_3225-4Pin_3.2x2.5mm_HandSoldering" H 2300 2000 50  0001 C CNN
 F 3 "~" H 2300 2000 50  0001 C CNN
 	1    2300 2000
@@
 F 0 "C6" V 1950 1750 50  0000 C CNN
 F 1 "22pF" V 1950 1950 50  0000 C CNN
-F 2 "" H 2100 1850 50  0001 C CNN
+F 2 "Capacitor_SMD:C_0805_2012Metric_Pad1.18x1.45mm_HandSolder" H 2100 1850 50  0001 C CNN
 F 3 "~" H 2100 1850 50  0001 C CNN
 	1    2100 1850
@@
 F 0 "C7" V 2200 2050 50  0000 C CNN
 F 1 "22pF" V 2200 2250 50  0000 C CNN
-F 2 "" H 2100 2150 50  0001 C CNN
+F 2 "Capacitor_SMD:C_0805_2012Metric_Pad1.18x1.45mm_HandSolder" H 2100 2150 50  0001 C CNN
 F 3 "~" H 2100 2150 50  0001 C CNN
 	1    2100 2150
@@
 F 0 "C8" V 1150 2550 50  0000 C CNN
 F 1 "0.1uF" V 1150 2750 50  0000 C CNN
-F 2 "" H 1050 2600 50  0001 C CNN
+F 2 "Capacitor_SMD:C_0805_2012Metric_Pad1.18x1.45mm_HandSolder" H 1050 2600 50  0001 C CNN
 F 3 "~" H 1050 2600 50  0001 C CNN
 	1    1050 2600
@@
 F 0 "R5" V 4450 3600 50  0000 C CNN
 F 1 "10k" V 4450 3750 50  0000 C CNN
-F 2 "" V 4390 3640 50  0001 C CNN
+F 2 "Resistor_SMD:R_0201_0603Metric" V 4390 3640 50  0001 C CNN
 F 3 "~" H 4350 3650 50  0001 C CNN
 	1    4350 3650
@@
 F 0 "R6" V 8250 5150 50  0000 L CNN
 F 1 "2.2k" V 8250 5300 50  0000 L CNN
-F 2 "" V 8390 5240 50  0001 C CNN
+F 2 "Resistor_SMD:R_0201_0603Metric" V 8390 5240 50  0001 C CNN
 F 3 "~" H 8350 5250 50  0001 C CNN
 	1    8350 5250
@@
 F 0 "R7" V 8450 5150 50  0000 L CNN
 F 1 "2.2k" V 8450 5300 50  0000 L CNN
-F 2 "" V 8590 5240 50  0001 C CNN
+F 2 "Resistor_SMD:R_0201_0603Metric" V 8590 5240 50  0001 C CNN
 F 3 "~" H 8550 5250 50  0001 C CNN
 	1    8550 5250
@@
 F 0 "R8" V 1150 1850 50  0000 C CNN
 F 1 "10k" V 1150 2000 50  0000 C CNN
-F 2 "" V 1090 1940 50  0001 C CNN
+F 2 "Resistor_SMD:R_0201_0603Metric" V 1090 1940 50  0001 C CNN
 F 3 "~" H 1050 1950 50  0001 C CNN
 	1    1050 1950
@@
 F 0 "J4" H 1257 7317 50  0000 C CNN
 F 1 "USB_C_Receptacle_USB2.0" H 1257 7226 50  0000 C CNN
-F 2 "" H 1300 6450 50  0001 C CNN
+F 2 "Connector_USB:USB_C_Receptacle_HRO_TYPE-C-31-M-12" H 1300 6450 50  0001 C CNN
 F 3 "https://www.usb.org/sites/default/files/documents/usb_type-c.zip" H 1300 6450 50  0001 C CNN
 	1    1150 6450
@@
 F 0 "R1" V 1800 5950 50  0000 C CNN
 F 1 "5.1K" V 1800 6100 50  0000 C CNN
-F 2 "" V 1940 6040 50  0001 C CNN
+F 2 "Resistor_SMD:R_0201_0603Metric" V 1940 6040 50  0001 C CNN
 F 3 "~" H 1900 6050 50  0001 C CNN
 	1    1900 6050
@@
 F 0 "R2" V 2000 6050 50  0000 C CNN
 F 1 "5.1K" V 2000 6200 50  0000 C CNN
-F 2 "" V 1940 6140 50  0001 C CNN
+F 2 "Resistor_SMD:R_0201_0603Metric" V 1940 6140 50  0001 C CNN
 F 3 "~" H 1900 6150 50  0001 C CNN
 	1    1900 6150
@@
 F 0 "F1" V 3850 7450 50  0000 C CNN
 F 1 "Polyfuse" V 4050 7300 50  0000 C CNN
-F 2 "" H 4000 7250 50  0001 L CNN
+F 2 "Fuse:Fuse_0603_1608Metric" H 4000 7250 50  0001 L CNN
 F 3 "~" H 3950 7450 50  0001 C CNN
 	1    3950 7450
@@
 F 0 "FB1" V 4100 7450 50  0000 C CNN
 F 1 "Ferrite_Bead" V 4350 7550 50  0000 C CNN
-F 2 "" V 4180 7450 50  0001 C CNN
+F 2 "Inductor_SMD:L_0201_0603Metric" V 4180 7450 50  0001 C CNN
 F 3 "~" H 4250 7450 50  0001 C CNN
 	1    4250 7450
