File: PCB/SofleKeyboard.kicad_pcb (KiCad board)
At the start: 2 copper layers, 137.2 x 109.2 mm, 87 parts, among them J1 LED, J2 4PIN, J3 OLED, P1 i2c_pin, P2 i2c_pin, SW1 SW_PUSH, SW10 SW_PUSH, SW11 SW_PUSH, SW12 SW_PUSH, SW13 SW_PUSH, SW14 SW_PUSH, SW15 SW_PUSH, SW16 SW_PUSH, SW17 SW_PUSH, SW18 SW_PUSH, SW19 SW_PUSH, SW2 SW_PUSH, SW20 SW_PUSH, SW21 SW_PUSH, SW22 SW_PUSH, SW23 SW_PUSH, SW24 SW_PUSH, SW25 Rotary_Encoder_Switch, SW26 SW_PUSH, SW27 SW_PUSH, SW28 SW_PUSH, SW29 SW_PUSH, SW3 SW_PUSH, SW30 SW_PUSH, SW4 SW_PUSH, SW5 SW_PUSH, SW6 SW_PUSH, SW7 SW_PUSH, SW8 SW_PUSH, SW9 SW_PUSH, U1 ProMicro

Commit message: Started PCB redux
Parts:
- added C1: 0.1uF, Capacitor_SMD:C_0805_2012Metric_Pad1.18x1.45mm_HandSolder, F.Cu at (118.1, 39.6)
- added C2: 0.1uF, Capacitor_SMD:C_0805_2012Metric_Pad1.18x1.45mm_HandSolder, F.Cu at (115.6, 39.6)
- added C3: 0.1uF, Capacitor_SMD:C_0805_2012Metric_Pad1.18x1.45mm_HandSolder, F.Cu at (113.0, 39.6)
- added C4: 0.1uF, Capacitor_SMD:C_0805_2012Metric_Pad1.18x1.45mm_HandSolder, F.Cu at (110.5, 39.6)
- added C5: 0.1uF, Capacitor_SMD:C_0805_2012Metric_Pad1.18x1.45mm_HandSolder, F.Cu at (105.4, 47.0)
- added C6: 22pF, Capacitor_SMD:C_0805_2012Metric_Pad1.18x1.45mm_HandSolder, F.Cu at (91.4, 59.7)
- added C7: 22pF, Capacitor_SMD:C_0805_2012Metric_Pad1.18x1.45mm_HandSolder, F.Cu at (91.4, 50.8)
- added C8: 0.1uF, Capacitor_SMD:C_0805_2012Metric_Pad1.18x1.45mm_HandSolder, F.Cu at (92.7, 79.0)
- added D31: PRTR5V0U2X, Package_TO_SOT_SMD:SOT-143, F.Cu at (92.7, 45.7)
- added F1: Polyfuse, Fuse:Fuse_0603_1608Metric, F.Cu at (96.5, 47.0)
- added FB1: Ferrite_Bead, Inductor_SMD:L_0201_0603Metric, F.Cu at (99.1, 47.0)
- added J4: USB_C_Receptacle_USB2.0, Connector_USB:USB_C_Receptacle_HRO_TYPE-C-31-M-12, F.Cu at (100.3, 40.6)
- added R1: 5.1K, Resistor_SMD:R_0201_0603Metric, F.Cu at (106.7, 43.2)
- added R2: 5.1K, Resistor_SMD:R_0201_0603Metric, F.Cu at (106.7, 41.9)
- added R3: 22, Resistor_SMD:R_0201_0603Metric, F.Cu at (100.3, 47.0)
- added R4: 22, Resistor_SMD:R_0201_0603Metric, F.Cu at (101.6, 47.0)
- added R5: 10k, Resistor_SMD:R_0201_0603Metric, F.Cu at (107.0, 63.5)
- added R6: 2.2k, Resistor_SMD:R_0201_0603Metric, F.Cu at (97.1, 64.9)
- added R7: 2.2k, Resistor_SMD:R_0201_0603Metric, F.Cu at (97.8, 64.9)
- added R8: 10k, Resistor_SMD:R_0201_0603Metric, F.Cu at (94.0, 50.5)
- added Y1: Crystal, Crystal:Crystal_SMD_3225-4Pin_3.2x2.5mm_HandSoldering, F.Cu at (91.6, 55.9)
- U1: value ProMicro -> ATmega32U4-AU; footprint SofleKeyboard-footprint:ProMicro -> Package_QFP:TQFP-44_10x10mm_P0.8mm
- moved U1 1.30 mm to (101.6, 57.1), turned to 270 degrees
Connections:
- net row0 renamed /row0
- net row1 renamed /row1
- net row2 renamed /row2
- net row3 renamed /row3
- D25 pad 1: row4 -> /row4
- D26 pad 1: row4 -> /row4
- D27 pad 1: row4 -> /row4
- D28 pad 1: row4 -> /row4
- D29 pad 1: row4 -> /row4
- D30 pad 1: row4 -> /row4
- J1 pad 2: LED -> /LED
- JP3 pad 2: SCL -> /SCL
- JP4 pad 2: SDA -> /SDA
- JP5 pad 2: SDA -> /SDA
- JP6 pad 2: SCL -> /SCL
- RSW1 pad 2: RESET -> /RESET
- SW10 pad 1: col2 -> /col2
- SW11 pad 1: col1 -> /col1
- SW12 pad 1: col0 -> /col0
- SW14 pad 1: col4 -> /col4
- SW15 pad 1: col3 -> /col3
- SW16 pad 1: col2 -> /col2
- SW17 pad 1: col1 -> /col1
- SW18 pad 1: col0 -> /col0
- SW2 pad 1: col4 -> /col4
- SW20 pad 1: col4 -> /col4
- SW21 pad 1: col3 -> /col3
- SW22 pad 1: col2 -> /col2
- SW23 pad 1: col1 -> /col1
- SW24 pad 1: col0 -> /col0
- SW25 pad A: ENCA -> /ENCA
- SW25 pad B: ENCB -> /ENCB
- SW26 pad 1: col4 -> /col4
- SW27 pad 1: col3 -> /col3
- SW28 pad 1: col2 -> /col2
- SW29 pad 1: col1 -> /col1
- SW3 pad 1: col3 -> /col3
- SW30 pad 1: col0 -> /col0
- SW4 pad 1: col2 -> /col2
- SW5 pad 1: col1 -> /col1
- SW6 pad 1: col0 -> /col0
- SW8 pad 1: col4 -> /col4
- SW9 pad 1: col3 -> /col3
- U1 pad 1: LED -> Net-(U1-Pad1)
- U1 pad 12: row4 -> /col2
- U1 pad 13: SW25A -> /RESET
- U1 pad 14: col4 -> VCC
- U1 pad 15: col3 -> GND
- U1 pad 16: col2 -> /XTAL2
- U1 pad 17: col1 -> /XTAL1
- U1 pad 18: col0 -> /SCL
- U1 pad 19: ENCB -> /SDA
- U1 pad 2: DATA -> VCC
- U1 pad 20: ENCA -> /DATA
- U1 pad 21: VCC -> /LED
- U1 pad 22: RESET -> Net-(U1-Pad22)
- U1 pad 24: Net-(U1-Pad24) -> VCC
- U1 pad 3: GND -> Net-(R4-Pad1)
- U1 pad 4: GND -> Net-(R3-Pad1)
- U1 pad 5: SDA -> GND
- U1 pad 6: SCL -> Net-(C5-Pad2)
- U1 pad 7: Net-(U1-Pad7) -> VCC
- W1 pad 1: DATA -> /DATA
Routing:
- net col0: track 358.0 -> 0.00 mm, vias 11 -> 0
- net col1: track 350.6 -> 0.00 mm, vias 11 -> 0
- net col2: track 334.4 -> 0.00 mm, vias 11 -> 0
- net col3: track 314.7 -> 0.00 mm, vias 11 -> 0
- net col4: track 311.0 -> 0.00 mm, vias 11 -> 0
- net /row3: track 170.1 -> 0.00 mm, vias 1 -> 0
- net /row2: track 165.8 -> 0.00 mm, vias 1 -> 0
- net row4: track 152.5 -> 0.00 mm, vias 1 -> 0
- net GND: track 124.4 -> 0.28 mm, vias 45 -> 0
- net ENCB: track 73.1 -> 0.00 mm, vias 1 -> 0
- net ENCA: track 69.0 -> 0.00 mm, vias 1 -> 0
- net VCC: track 74.2 -> 15.5 mm, vias 3 -> 0
- net SDA: track 57.0 -> 0.00 mm, vias 4 -> 0
- net LED: track 55.8 -> 0.00 mm, vias 1 -> 0
- net RESET: track 51.2 -> 0.00 mm
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- removed copper zone on B.Cu, net GND
- removed copper zone on F.Cu, net GND
